Commit message: Updated URDF for better visibility

File: hand_description/urdf/underactuated_hand_urdf.urdf (robot description, URDF)
Before this commit: robot hand_description, 9 links, 8 joints
Joints:
- joint finger1_dist_joint: axis -1 0 0 -> 1 0 0; limit lower=-1.57 upper=1.57 effort=0 velocity=0 -> lower=0 upper=1.57 effort=0 velocity=0
- joint finger1_prox_joint: axis -1 0 0 -> 1 0 0; limit lower=-1.57 upper=1.57 effort=0 velocity=0 -> lower=0 upper=1.57 effort=0 velocity=0
- joint finger1_roll_joint: axis 0 -1 0 -> 0 1 0; limit lower=-1.57 upper=1.57 effort=0 velocity=0 -> lower=0 upper=1.57 effort=0 velocity=0
- joint finger2_dist_joint: limit lower=-1.57 upper=1.57 effort=0 velocity=0 -> lower=0 upper=1.57 effort=0 velocity=0
- joint finger2_prox_joint: axis 1 0 0 -> -1 0 0; limit lower=-1.57 upper=1.57 effort=0 velocity=0 -> lower=0 upper=1.57 effort=0 velocity=0
- joint finger2_roll_joint: limit lower=-1.57 upper=1.57 effort=0 velocity=0 -> lower=0 upper=1.57 effort=0 velocity=0; origin xyz=0.028 0.035 0.068 rpy=1.5708 0 2.4435 -> xyz=0.028 0.035 0.068 rpy=1.5708 0 3.142
- joint thumb_dist_joint: axis -1 0 0 -> 1 0 0; limit lower=-1.57 upper=1.57 effort=0 velocity=0 -> lower=0 upper=1.57 effort=0 velocity=0
- joint thumb_prox_joint: axis -1 0 0 -> 1 0 0; limit lower=-1.57 upper=1.57 effort=0 velocity=0 -> lower=0 upper=1.57 effort=0 velocity=0
